File: design_files/ASM2101.brd (EAGLE design)
At the start: 16.5 x 16.5 mm, 19 parts, among them J1 GRPB032VWQS, J2 GRPB051VWCN, U1 ATMEGA328P-MU

Commit message: update format
Parts:
- moved C2 18.4 mm to (25.0, 17.4)
- moved U$11 18.4 mm to (19.5, 13.4)
- moved U$12 18.4 mm to (19.5, 24.6)
- moved U$2 18.4 mm to (15.4, 17.5)
- moved U$9 18.4 mm to (26.6, 17.5)
- moved $1 18.4 mm to (26.6, 20.5)
- moved C1 18.4 mm to (17.5, 20.7)
- moved C3 18.4 mm to (24.7, 21.0)
- moved J1 18.4 mm to (20.3, 20.1)
- moved J2 18.4 mm to (21.0, 17.2)
- moved U$1 18.4 mm to (16.9, 14.9)
- moved U$10 18.4 mm to (25.1, 14.9)
- moved U$3 18.4 mm to (15.4, 20.5)
- moved U$4 18.4 mm to (16.9, 23.1)
- moved U$5 18.4 mm to (25.1, 23.1)
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Routing:
- net AD0: track 9.15 -> 8.10 mm
Other:
- board size 16.5 x 16.5 mm -> 19.1 x 19.1 mm
- board text added: "4"
- board text added: "Rev4"
- board text added: "TinyCircuits.com"
- board text removed: "REV 3"
- board text removed: "Tiny-Circuits.com"
